File: hardware/rev0.1/ProgramMemory_sch.kicad_sch (KiCad schematic)
At the start: 16 parts, among them U13 74LS02, U14 2716, U15 6116, U16 6116, U17 74LS00, U18 74LS541, U19 4289_MEMORY_IF

Commit message: Initial commit
Connections:
- net at U15.21 (~{WE}): now also U17.3; no longer U17.6
- net at U16.21 (~{WE}): now also U17.6; no longer U17.3
Changed lines of the file:
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@@
-    (stroke (width 0) (type default) (color 0 0 0 0))
-  )
-  (wire (pts (xy 199.39 30.48) (xy 199.39 39.37))
     (stroke (width 0) (type default) (color 0 0 0 0))
   )
@@
     (stroke (width 0) (type default) (color 0 0 0 0))
   )
-  (wire (pts (xy 179.07 30.48) (xy 199.39 30.48))
+  (wire (pts (xy 179.07 30.48) (xy 237.49 30.48))
     (stroke (width 0) (type default) (color 0 0 0 0))
   )
@@
     (stroke (width 0) (type default) (color 0 0 0 0))
   )
+  (wire (pts (xy 237.49 30.48) (xy 237.49 39.37))
+    (stroke (width 0) (type default) (color 0 0 0 0))
+  )
   (wire (pts (xy 92.71 39.37) (xy 92.71 27.94))
     (stroke (width 0) (type default) (color 0 0 0 0))
@@
     (stroke (width 0) (type default) (color 0 0 0 0))
   )
+  (wire (pts (xy 199.39 33.02) (xy 199.39 39.37))
+    (stroke (width 0) (type default) (color 0 0 0 0))
+  )
   (wire (pts (xy 158.75 21.59) (xy 207.01 21.59))
     (stroke (width 0) (type default) (color 0 0 0 0))
@@
     (stroke (width 0) (type default) (color 0 0 0 0))
   )
-  (wire (pts (xy 237.49 33.02) (xy 237.49 39.37))
-    (stroke (width 0) (type default) (color 0 0 0 0))
-  )
   (wire (pts (xy 43.18 154.94) (xy 59.69 154.94))
     (stroke (width 0) (type default) (color 0 0 0 0))
@@
     (stroke (width 0) (type default) (color 0 0 0 0))
   )
-  (wire (pts (xy 181.61 33.02) (xy 237.49 33.02))
-    (stroke (width 0) (type default) (color 0 0 0 0))
-  )
   (wire (pts (xy 234.95 64.77) (xy 234.95 77.47))
     (stroke (width 0) (type default) (color 0 0 0 0))
@@
     (stroke (width 0) (type default) (color 0 0 0 0))
   )
+  (wire (pts (xy 181.61 33.02) (xy 199.39 33.02))
+    (stroke (width 0) (type default) (color 0 0 0 0))
+  )
   (wire (pts (xy 123.19 88.9) (xy 123.19 189.23))
     (stroke (width 0) (type default) (color 0 0 0 0))
@@
     (stroke (width 0) (type default) (color 0 0 0 0))
   )
-  (text "~{WE}(OPR)" (at 171.45 125.73 0)
+  (text "~{WE}(OPA)" (at 171.45 125.73 0)
     (effects (font (size 1.27 1.27)) (justify left bottom))
   )
@@
     (effects (font (size 1.27 1.27)) (justify left bottom))
   )
-  (text "~{WE}(OPA)" (at 171.45 116.84 0)
+  (text "~{WE}(OPR)" (at 171.45 116.84 0)
     (effects (font (size 1.27 1.27)) (justify left bottom))
   )
